Commit message: Added inertial_macros

File: description/robot_core.xacro (robot description, xacro)
@@ -1,4 +1,5 @@
 <?xml version="1.0"?>
 <robot xmlns:xacro="http://www.ros.org/wiki/xacro">
+<xacro:include filename = "inertial_macros.xacro"/>
 <material name = "white">
     <color rgba = "1 1 1 1"/>
@@ -14,6 +15,5 @@
 </material>
 <!--BASE LINK -->
-<link name = "base_link">
-</link>
+<link name = "base_link"/>
 <!--CHASSIS JOINT -->
 <joint name = "chassis_joint" type="fixed">
@@ -31,12 +31,22 @@
         <material name ="white"/>
     </visual>
+    <collision>
+        <origin xyz = "0.15 0 0.075"/>
+        <geometry>
+            <box size = "0.3 0.3 0.15"/>
+        </geometry>
+    </collision>
+    <xacro:inertial_box mass ="0.5" x ="0.3" y="0.3" z="0.15">
+        <origin xyz = "0.15 0 0.075" rpy ="0 0 0"/>
+    </xacro:inertial_box>
 </link>
-<!-- LEFT WHEEL -->
-<joint name="left_wheel_joint" type="continious">
+<!-- LEFT WHEEL Joint-->
+<joint name="left_wheel_joint" type="continuous">
     <parent link = "base_link"/>
     <child link = "left_wheel"/>
-    <origin xyz="0 0.175 0" rpy="-$(pi/2) 0 0"/>
+    <origin xyz="0 0.175 0" rpy="-${pi/2} 0 0"/>
     <axis xyz = "0 0 1" />
 </joint>
+<!-- LEFT WHEEL Link-->
 <link name="left_wheel">
     <visual>
@@ -45,10 +55,19 @@
         </geometry>
         <material name="blue"/>
+    </visual>
+    <collision>
+        <geometry>
+            <cylinder radius = "0.05" length="0.04"/>
+        </geometry>
+    </collision>
+    <xacro:inertial_cylinder mass= "0.1" length= "0.04" radius= "0.05">
+        <origin xyz="0 0 0" rpy="0 0 0"/>
+    </xacro:inertial_cylinder>
 </link>
 <!-- RIGHT WHEEL -->
-<joint name="right_wheel_joint" type="continious">
+<joint name="right_wheel_joint" type="continuous">
     <parent link = "base_link"/>
     <child link = "right_wheel"/>
-    <origin xyz="0 -0.175 0" rpy="$(pi/2) 0 0"/>
+    <origin xyz="0 -0.175 0" rpy="${pi/2} 0 0"/>
     <axis xyz = "0 0 -1" />
 </joint>
@@ -59,4 +78,35 @@
         </geometry>
         <material name="blue"/>
+    </visual>
+    <collision>
+        <geometry>
+            <cylinder radius = "0.05" length="0.04"/>
+        </geometry>
+    </collision>
+    <xacro:inertial_cylinder mass= "0.1" length="0.05" radius= "0.04">
+        <origin xyz="0 0 0" rpy="0 0 0"/>
+    </xacro:inertial_cylinder>
+</link>
+<!--CASTER WHEEL -->
+<joint name = "caster_wheel_joint" type = "fixed">
+    <parent link = "chassis"/>
+    <child link = "caster_wheel"/>
+    <origin xyz = "0.24 0 0"/>
+</joint>
+<link name="caster_wheel">
+    <visual>
+        <geometry>
+            <sphere radius = "0.05" />
+            <material name = "black"/>
+        </geometry>
+    </visual>
+    <collision>
+        <geometry>
+            <sphere radius = "0.05" />
+        </geometry>
+    </collision>
+    <xacro:inertial_sphere mass= "0.1" radius= "0.05">
+        <origin xyz="0 0 0" rpy="0 0 0"/>
+    </xacro:inertial_sphere>
 </link>
 </robot>
